Commit message: Added 2 links and a joint

File: src/my_robot/robot.urdf (robot description, URDF)
Before this commit: robot robot, 1 links, 0 joints
Links:
- added link second_link; visual cylinder length=0.2 radius=0.1
Joints:
- added joint base_second: type fixed, parent base_link, child second_link, origin xyz=0.0 0.0 0.2 rpy=0.0 0.0 0.0

Commit message: Added revolute joint

File: src/my_robot/robot.urdf (robot description, URDF)
Before this commit: robot robot, 2 links, 1 joints
Joints:
- joint base_second: axis (none) -> 0.0 0.0 1.0; limit (none) -> lower=-1.57 upper=1.57 effort=100.0 velocity=100.0; type fixed -> revolute

Commit message: Wrote urdf for a simple two wheeled robot

File: src/my_robot/robot.urdf (robot description, URDF)
Before this commit: robot robot, 2 links, 1 joints
Links:
- removed link second_link
- added link base_footprint
- added link castor; visual sphere radius=0.05
- added link left_wheel; visual cylinder length=0.05 radius=0.1
- added link right_wheel; visual cylinder length=0.05 radius=0.1
Joints:
- removed joint base_second
- added joint base_footprint_to_base_link: type fixed, parent base_footprint, child base_link, origin xyz=0.0 0.0 0.1 rpy=0.0 0.0 0.0
- added joint base_link_to_castor: type fixed, parent base_link, child castor, origin xyz=0.2 0.0 -0.05 rpy=0.0 0.0 0.0
- added joint base_link_to_left_wheel: type continuous, parent base_link, child left_wheel, origin xyz=-0.15 0.225 0.0 rpy=0.0 0.0 0.0, axis 0.0 1.0 0.0
- added joint base_link_to_right_wheel: type continuous, parent base_link, child right_wheel, origin xyz=-0.15 -0.225 0.0 rpy=0.0 0.0 0.0, axis 0.0 1.0 0.0
