Commit message: Learnt about and used xacro variable

File: src/my_robot_two_wheel/urdf/robot.urdf.xacro (robot description, xacro)
@@ -34,4 +34,5 @@
 </robot> -->
 <robot name="two_wheeled_robot" xmlns:xacro="https://www.ros.org/wiki/xacro">
+    <xacro:property name="base_length" value="0.6" />
     <link name="base_footprint">
         <origin xyz="0.0 0.0 0.0" rpy="0.0 0.0 0.0" />
@@ -41,5 +42,5 @@
             <origin xyz="0.0 0.0 0.1" rpy="0.0 0.0 0.0" />
             <geometry>
-                <box size="0.6 0.4 0.2" />
+                <box size="${base_length} 0.4 0.2" />
             </geometry>
             <material name="">
@@ -55,5 +56,5 @@
     <link name="left_wheel">
         <visual name="">
-            <origin xyz="0.0 0.0 0.0" rpy="1.57 0.0 0.0" />
+            <origin xyz="0.0 0.0 0.0" rpy="${pi / 2.0} 0.0 0.0" />
             <geometry>
                 <cylinder radius="0.1" length="0.05" />
@@ -64,5 +65,5 @@
     <link name="right_wheel">
         <visual name="">
-            <origin xyz="0.0 0.0 0.0" rpy="1.57 0.0 0.0" />
+            <origin xyz="0.0 0.0 0.0" rpy="${pi / 2.0} 0.0 0.0" />
             <geometry>
                 <cylinder radius="0.1" length="0.05" />
@@ -93,5 +94,5 @@
     </joint>
     <joint name="base_link_to_right_wheel" type="continuous">
-        <origin xyz="-0.15 -0.225 0.0" rpy="0.0 0.0 0.0" />
+        <origin xyz="${-base_length / 4.0} -0.225 0.0" rpy="0.0 0.0 0.0" />
         <parent link="base_link" />
         <child link="right_wheel" />

Commit message: Learnt to use xacro-macros

File: src/my_robot_two_wheel/urdf/robot.urdf.xacro (robot description, xacro)
@@ -35,4 +35,13 @@
 <robot name="two_wheeled_robot" xmlns:xacro="https://www.ros.org/wiki/xacro">
     <xacro:property name="base_length" value="0.6" />
+    <xacro:macro name="wheels" params="roll radius length material">
+        <visual name="">
+            <origin xyz="0.0 0.0 0.0" rpy="${roll} 0.0 0.0" />
+            <geometry>
+                <cylinder radius="${radius}" length="${length}" />
+            </geometry>
+            <material name="${material}" />
+        </visual>
+    </xacro:macro>
     <link name="base_footprint">
         <origin xyz="0.0 0.0 0.0" rpy="0.0 0.0 0.0" />
@@ -55,5 +64,5 @@
     </material>
     <link name="left_wheel">
-        <visual name="">
+        <!-- <visual name="">
             <origin xyz="0.0 0.0 0.0" rpy="${pi / 2.0} 0.0 0.0" />
             <geometry>
@@ -61,5 +70,6 @@
             </geometry>
             <material name="grey" />
-        </visual>
+        </visual> -->
+        <xacro:wheels roll="${pi/2.0}" radius="0.1" length="0.05" material="grey" />
     </link>
     <link name="right_wheel">
