Commit message: Changed the root_base_link joint origin (Shifted base link wrt root in order to keep root on ground and bot above ground)

File: src/differential_drive_bot/urdf/differential_drive_bot.urdf (robot description, URDF)
Before this commit: robot differential_drive_bot, 11 links, 10 joints
Joints:
- joint fixed_node_to_root_joint: origin xyz=0.3 0.2 -0.075 rpy=0 -0 0 -> xyz=0 0 0.05 rpy=0 -0 0

Commit message: Added a separate package for launching the bot

File: src/differential_drive_bot/urdf/differential_drive_bot.urdf (robot description, URDF)
Before this commit: robot differential_drive_bot, 11 links, 10 joints
Links:
- link castor_holder_castor: mass None -> 0.001
- link castor_holder_castor_1: mass None -> 0.001
Joints:
- removed joint castor_holder_castor
- removed joint castor_holder_castor_1
- removed joint castor_holder_castor_2
- added joint castor_holder_castor_1j: type continuous, parent castor_holder_castor_1, child castor_holder_castor, origin xyz=0 0 0 rpy=0 -0 0, axis 0 1 0
- added joint castor_holder_castor_2j: type continuous, parent castor_holder_castor, child castor, origin xyz=0 0 0 rpy=0 -0 0, axis 0 0 1
- added joint castor_holder_castor_j: type continuous, parent castor_holder, child castor_holder_castor_1, origin xyz=0 -2.92793e-17 -0.025 rpy=0 -0 0, axis 1 0 0
