Commit message: Added gazebo plugins to move the wheels and arms along with gazebo bridge

File: src/differential_drive_bot/urdf/differential_drive_bot.urdf.xacro (robot description, xacro)
@@ -130,32 +130,6 @@
         </visual>
     </link>
-    <link name="castor_holder_castor">
-        <inertial>
-            <origin xyz="0 0 0" rpy="0 0 0" />
-            <mass value="0.001" />
-            <inertia
-                ixx="1e-6"
-                ixy="0"
-                ixz="0"
-                iyy="1e-6"
-                iyz="0"
-                izz="1e-6" />
-        </inertial>
-    </link>
-    <link name="castor_holder_castor_1">
-        <inertial>
-            <origin xyz="0 0 0" rpy="0 0 0" />
-            <mass value="0.001" />
-            <inertia
-                ixx="1e-6"
-                ixy="0"
-                ixz="0"
-                iyy="1e-6"
-                iyz="0"
-                izz="1e-6" />
-        </inertial>
-    </link>
     <link name="root" />
-    <link name="wheel">
+    <link name="wheel_left">
         <inertial>
             <mass value="0.981748" />
@@ -166,5 +140,6 @@
             <origin xyz="0 0 0" rpy="0 -0 0" />
             <geometry>
-                <mesh filename="package://differential_drive_bot/meshes/wheel.stl" scale="1 1 1" />
+                <mesh filename="package://differential_drive_bot/meshes/wheel_left.stl"
+                    scale="1 1 1" />
             </geometry>
             <material name="0.647059_0.647059_0.647059_0.000000_0.000000">
@@ -174,14 +149,15 @@
         <xacro:sphere_collision radius="${wheel_radius}" z="${wheel_z}" />
     </link>
-    <link name="wheel_1">
+    <link name="wheel_right">
         <inertial>
             <mass value="0.981748" />
-            <origin xyz="-1.94909e-18 6.12323e-18 0.0125" rpy="0 -0 0" />
+            <origin xyz="-1.94909e-18 4.62223e-33 0.0125" rpy="0 -0 0" />
             <inertia ixx="0.0025055" ixy="0" ixz="0" iyy="0.0025055" iyz="0" izz="0.00490874" />
         </inertial>
         <visual>
-            <origin xyz="0 0 0" rpy="0 -0 0" />
-            <geometry>
-                <mesh filename="package://differential_drive_bot/meshes/wheel.stl" scale="1 1 1" />
+            <origin xyz="0 -6.12323e-18 0" rpy="0 -0 0" />
+            <geometry>
+                <mesh filename="package://differential_drive_bot/meshes/wheel_right.stl"
+                    scale="1 1 1" />
             </geometry>
             <material name="0.647059_0.647059_0.647059_0.000000_0.000000">
@@ -196,5 +172,6 @@
         <parent link="arm_1" />
         <child link="arm" />
-        <limit effort="1" velocity="1" lower="-2.61799" upper="2.61799" />
+        <limit effort="100" velocity="100" lower="-2.61799" upper="2.61799" />
+        <dynamics friction="0.3" damping="0.3" />
     </joint>
     <joint name="arm_mount_arm_1" type="revolute">
@@ -203,5 +180,6 @@
         <parent link="arm_mount" />
         <child link="arm_1" />
-        <limit effort="1" velocity="1" lower="-1.5708" upper="1.5708" />
+        <limit effort="100" velocity="100" lower="-1.5708" upper="1.5708" />
+        <dynamics friction="0.3" damping="0.3" />
     </joint>
     <joint name="base_link_arm_mount" type="fixed">
@@ -212,5 +190,5 @@
     </joint>
     <joint name="base_link_castor_holder" type="fixed">
-        <origin xyz="-0.12 -0.2 -1.38778e-17" rpy="0 -0 0" />
+        <origin xyz="-0.12 -0.2 0" rpy="8.32667e-17 -0 3.14159" />
         <axis xyz="0 0 1" />
         <parent link="base_link" />
@@ -221,32 +199,20 @@
         <axis xyz="0 0 1" />
         <parent link="base_link" />
-        <child link="wheel" />
+        <child link="wheel_left" />
     </joint>
     <joint name="base_link_wheel_2" type="continuous">
         <origin xyz="-0.5 -0.4 0.05" rpy="1.5708 6.16298e-33 9.25186e-17" />
-        <axis xyz="0 0 1" />
-        <parent link="base_link" />
-        <child link="wheel_1" />
-    </joint>
-    <joint name="castor_holder_castor_j" type="continuous">
-        <origin xyz="0 -2.92793e-17 -0.025" rpy="0 -0 0" />
-        <axis xyz="1 0 0" />
+        <axis xyz="0 0 -1" />
+        <parent link="base_link" />
+        <child link="wheel_right" />
+    </joint>
+    <joint name="castor_holder_castor" type="fixed">
+        <origin xyz="0 0 -0.025" rpy="0 -0 0" />
+        <axis xyz="0 0 1" />
         <parent link="castor_holder" />
-        <child link="castor_holder_castor_1" />
-    </joint>
-    <joint name="castor_holder_castor_1j" type="continuous">
-        <origin xyz="0 0 0" rpy="0 -0 0" />
-        <axis xyz="0 1 0" />
-        <parent link="castor_holder_castor_1" />
-        <child link="castor_holder_castor" />
-    </joint>
-    <joint name="castor_holder_castor_2j" type="continuous">
-        <origin xyz="0 0 0" rpy="0 -0 0" />
-        <axis xyz="0 0 1" />
-        <parent link="castor_holder_castor" />
         <child link="castor" />
     </joint>
     <joint name="fixed_node_to_root_joint" type="fixed">
-        <origin xyz="0 0 0.05" rpy="0 -0 0" />
+        <origin xyz="0.3 0.2 0.05" rpy="0 -0 0" />
         <axis xyz="0 0 1" />
         <parent link="root" />
@@ -254,4 +220,8 @@
     </joint>
     <!-- GAZEBO PLUGINS -->
+    <gazebo reference="castor">
+        <mu1 value="0.1" />
+        <mu2 value="0.1" />
+    </gazebo>
     <gazebo>
         <plugin
@@ -260,8 +230,24 @@
             <left_joint>base_link_wheel_1</left_joint>
             <right_joint>base_link_wheel_2</right_joint>
-            <wheel_separation>0.45</wheel_separation>
+            <wheel_separation>0.4</wheel_separation>
             <wheel_radius>0.1</wheel_radius>
             <frame_id>odom</frame_id>
             <child_frame_id>root</child_frame_id>
+        </plugin>
+    </gazebo>
+    <gazebo>
+        <plugin
+            filename="gz-sim-joint-position-controller-system"
+            name="gz::sim::systems::JointPositionController">
+            <joint_name>arm_mount_arm_1</joint_name>
+            <p_gain>5.0</p_gain>
+        </plugin>
+    </gazebo>
+    <gazebo>
+        <plugin
+            filename="gz-sim-joint-position-controller-system"
+            name="gz::sim::systems::JointPositionController">
+            <joint_name>arm_1_arm_2</joint_name>
+            <p_gain>3.0</p_gain>
         </plugin>
     </gazebo>
@@ -272,4 +258,6 @@
             <joint_name>base_link_wheel_1</joint_name>
             <joint_name>base_link_wheel_2</joint_name>
+            <joint_name>arm_mount_arm_1</joint_name>
+            <joint_name>arm_1_arm_2</joint_name>
         </plugin>
     </gazebo>

Commit message: Added camera link

File: src/differential_drive_bot/urdf/differential_drive_bot.urdf.xacro (robot description, xacro)
@@ -4,4 +4,7 @@
     <xacro:property name="base_link_b" value="0.4" />
     <xacro:property name="base_link_h" value="${0.15+0.03}" />
+    <xacro:property name="camera_l" value="0.1" />
+    <xacro:property name="camera_b" value="0.07" />
+    <xacro:property name="camera_h" value="0.05" />
     <xacro:property name="arm_l" value="0.02" />
     <xacro:property name="arm_b" value="0.05" />
@@ -96,4 +99,22 @@
             x="${-base_link_l/2}" y="${-base_link_b/2}" z="${(base_link_h/2) - 0.025}" />
     </link>
+    <link name="camera">
+        <inertial>
+            <mass value="0.1675" />
+            <origin xyz="-6.99007e-18 1.59925e-18 0.025" rpy="0 -0 0" />
+            <inertia ixx="0.000152792" ixy="0" ixz="0" iyy="0.000237479" iyz="0" izz="0.000279979" />
+        </inertial>
+        <visual>
+            <origin xyz="-8.57036e-18 8.67362e-19 0" rpy="0 -0 0" />
+            <geometry>
+                <mesh filename="package://differential_drive_bot/meshes/camera.stl" scale="1 1 1" />
+            </geometry>
+            <material name="0.980392_0.713725_0.003922_0.000000_0.000000">
+                <color rgba="0.980392 0.713726 0.00392157 1" />
+            </material>
+        </visual>
+        <xacro:box_collision l="${camera_l}" b="${camera_b}" h="${camera_h}"
+            x="${0}" y="${0}" z="${camera_h/2}" />
+    </link>
     <link name="castor">
         <inertial>
@@ -212,4 +233,10 @@
         <parent link="castor_holder" />
         <child link="castor" />
+    </joint>
+    <joint name="base_link_camera" type="fixed">
+        <origin xyz="0 -0.2 0.05" rpy="1.5708 -0 1.5708" />
+        <axis xyz="0 0 1" />
+        <parent link="base_link" />
+        <child link="camera" />
     </joint>
     <joint name="fixed_node_to_root_joint" type="fixed">

Commit message: Added gazebo world

File: src/differential_drive_bot/urdf/differential_drive_bot.urdf.xacro (robot description, xacro)
@@ -99,5 +99,5 @@
             x="${-base_link_l/2}" y="${-base_link_b/2}" z="${(base_link_h/2) - 0.025}" />
     </link>
-    <link name="camera">
+    <link name="camera_link">
         <inertial>
             <mass value="0.1675" />
@@ -238,5 +238,5 @@
         <axis xyz="0 0 1" />
         <parent link="base_link" />
-        <child link="camera" />
+        <child link="camera_link" />
     </joint>
     <joint name="fixed_node_to_root_joint" type="fixed">
@@ -289,3 +289,30 @@
         </plugin>
     </gazebo>
+    <gazebo reference="camera_link">
+        <sensor name="camera" type="camera">
+            <camera>
+                <horizontal_fov>1.3962634</horizontal_fov>
+                <image>
+                    <width>640</width>
+                    <height>480</height>
+                    <format>R8G8B8</format>
+                </image>
+                <clip>
+                    <near>0.1</near>
+                    <far>15</far>
+                </clip>
+                <noise>
+                    <type>gaussian</type>
+                    <mean>0.0</mean>
+                    <stddev>0.007</stddev>
+                </noise>
+                <optical_frame_id>camera_link</optical_frame_id>
+                <camera_info_topic>camera/camera_info</camera_info_topic>
+            </camera>
+            <always_on>1</always_on>
+            <update_rate>20</update_rate>
+            <visualize>true</visualize>
+            <topic>camera/image_raw</topic>
+        </sensor>
+    </gazebo>
 </robot>

Commit message: Integrated camera

File: src/differential_drive_bot/urdf/differential_drive_bot.urdf.xacro (robot description, xacro)
@@ -106,7 +106,8 @@
         </inertial>
         <visual>
-            <origin xyz="-8.57036e-18 8.67362e-19 0" rpy="0 -0 0" />
-            <geometry>
-                <mesh filename="package://differential_drive_bot/meshes/camera.stl" scale="1 1 1" />
+            <origin xyz="0 0 0" rpy="0 -0 0" />
+            <geometry>
+                <!-- <mesh filename="package://differential_drive_bot/meshes/camera.stl" scale="1 1 1" /> -->
+                <box size="${0.05} ${0.1} ${camera_h}"/>
             </geometry>
             <material name="0.980392_0.713725_0.003922_0.000000_0.000000">
@@ -114,5 +115,5 @@
             </material>
         </visual>
-        <xacro:box_collision l="${camera_l}" b="${camera_b}" h="${camera_h}"
+        <xacro:box_collision l="${0.05}" b="${0.1}" h="${camera_h}"
             x="${0}" y="${0}" z="${camera_h/2}" />
     </link>
@@ -235,6 +236,6 @@
     </joint>
     <joint name="base_link_camera" type="fixed">
-        <origin xyz="0 -0.2 0.05" rpy="1.5708 -0 1.5708" />
-        <axis xyz="0 0 1" />
+        <origin xyz="0.025 -0.2 0.05" rpy="${0} -0 ${0}" />
+        <!-- <axis xyz="0 0 1" /> -->
         <parent link="base_link" />
         <child link="camera_link" />
@@ -245,4 +246,15 @@
         <parent link="root" />
         <child link="base_link" />
+    </joint>
+    <!-- Camera OPEN CV SETUP -->
+    <link name="camera_link_optical">
+    </link>
+    <joint name="camera_optical_joint" type="fixed">
+        <!-- these values have to be these values otherwise the gazebo camera
+        image won't be aligned properly with the frame it is supposedly
+        originating from -->
+        <origin xyz="0 0 0" rpy="${-pi/2} 0 ${-pi/2}" />
+        <parent link="camera_link" />
+        <child link="camera_link_optical" />
     </joint>
     <!-- GAZEBO PLUGINS -->
@@ -307,5 +319,5 @@
                     <stddev>0.007</stddev>
                 </noise>
-                <optical_frame_id>camera_link</optical_frame_id>
+                <optical_frame_id>camera_link_optical</optical_frame_id>
                 <camera_info_topic>camera/camera_info</camera_info_topic>
             </camera>
